File: schematic/tanguito/tanguito.kicad_sch (KiCad schematic)
At the start: 14 parts, among them J1 Barrel_Jack, M1 DC Motor 12V, M2 DC Motor 12V, M3 DC Motor 12V, U1 MP1584_Module, U2 L298N, U3 L298N

Commit message: pcb: updated
Parts:
- U2: footprint Connector_PinHeader_2.54mm:PinHeader_1x10_P2.54mm_Vertical -> Connector_PinHeader_2.54mm:PinHeader_1x12_P2.54mm_Vertical
Connections:
- net PWM3: now also U2.9 (EnA); no longer U2.11 (EnB)
- net PWM4: now also U2.11 (EnB); no longer U3.6 (EnA)
- net GPIO7: now reaches P2.38 (GPIO7)
- net GPIO7: now also U3.5 (IN1)
- net ENET_RXD1: now reaches P2.4 (RXD1)
- net ENET_RXD1: now also A1.15 (STEP)
- net GPIO8: now reaches P2.40 (GPIO8)
- net GPIO8: now also U3.6 (EnA)
- net ENET_TXEN: now reaches P2.6 (TX_EN)
- net ENET_TXEN: now also A1.16 (DIR)
- net T_FIL0: now reaches P1.33 (T_FL0)
- net T_FIL0: now also U2.12 (IN4)
- net T_COL0: now reaches P1.39 (T_COL0)
- net T_COL0: now also U2.7 (IN1)
- net GPIO0: no longer names the net of P2.29 (GPIO0)
- net GPIO0: no longer U2.7 (IN1)
- net GPIO1: no longer names the net of P2.32 (GPIO1)
- net GPIO1: no longer U2.12 (IN4)
- net GPIO2: no longer names the net of P2.31 (GPIO2)
- net GPIO2: no longer A1.15 (STEP)
- net GPIO3: no longer names the net of P2.34 (GPIO3)
- net GPIO3: no longer A1.16 (DIR)
- net GPIO4: no longer names the net of P2.33 (GPIO4)
- net GPIO4: no longer U3.5 (IN1)
- net PWM0: no longer names the net of P1.36 (T_FL1)
- net PWM0: no longer U2.9 (EnA)
Changed lines of the file:
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@@
 	(wire
 		(pts
-			(xy 57.15 50.8) (xy 50.8 50.8)
-		)
-		(stroke
-			(width 0)
-			(type default)
-		)
-	)
-	(wire
-		(pts
 			(xy 254 148.59) (xy 260.35 148.59)
 		)
@@
 	(wire
 		(pts
-			(xy 57.15 45.72) (xy 50.8 45.72)
-		)
-		(stroke
-			(width 0)
-			(type default)
-		)
-	)
-	(wire
-		(pts
 			(xy 195.58 78.74) (xy 194.31 78.74)
 		)
@@
 	(wire
 		(pts
-			(xy 57.15 43.18) (xy 50.8 43.18)
-		)
-		(stroke
-			(width 0)
-			(type default)
-		)
-	)
-	(wire
-		(pts
 			(xy 20.32 27.94) (xy 25.4 27.94)
 		)
@@
 	(wire
 		(pts
-			(xy 50.8 40.64) (xy 57.15 40.64)
-		)
-		(stroke
-			(width 0)
-			(type default)
-		)
-	)
-	(wire
-		(pts
 			(xy 99.06 30.48) (xy 105.41 30.48)
 		)
@@
 	(wire
 		(pts
-			(xy 57.15 38.1) (xy 50.8 38.1)
-		)
-		(stroke
-			(width 0)
-			(type default)
-		)
-	)
-	(wire
-		(pts
 			(xy 194.31 71.12) (xy 194.31 78.74)
 		)
@@
 	(wire
 		(pts
-			(xy 99.06 33.02) (xy 100.33 33.02)
-		)
-		(stroke
-			(width 0)
-			(type default)
-		)
-	)
-	(wire
-		(pts
 			(xy 153.67 59.69) (xy 153.67 57.15)
 		)
@@
 		)
 	)
+		(label "ENET_RXD1"
+		(at 25.4 30.48 180)
+		(effects
+			(font
+				(size 1.27 1.27)
+			)
+			(justify right bottom)
+		)
+	)
+	(label "ENET_TXEN"
+		(at 25.4 35.56 180)
+		(effects
+			(font
+				(size 1.27 1.27)
+			)
+			(justify right bottom)
+		)
+	)
+	(label "GPIO7"
+		(at 50.8 27.94 0)
+		(effects
+			(font
+				(size 1.27 1.27)
+			)
+			(justify left bottom)
+		)
+	)
+	(label "GPIO8"
+		(at 50.8 22.86 0)
+		(effects
+			(font
+				(size 1.27 1.27)
+			)
+			(justify left bottom)
+		)
+	)
+	(label "T_FIL0"
+		(at 99.06 40.64 0)
+		(effects
+			(font
+				(size 1.27 1.27)
+			)
+			(justify left bottom)
+		)
+	)
+	(label "T_COL0"
+		(at 99.06 25.4 0)
+		(effects
+			(font
+				(size 1.27 1.27)
+			)
+			(justify left bottom)
+		)
+	)
 	(label "M2-"
 		(at 224.79 43.18 0)
@@
 		)
 	)
-	(label "PWM4"
+	(label "GPIO8"
 		(at 186.69 134.62 0)
 		(effects
@@
 		)
 	)
-	(label "GPIO1"
+	(label "T_FIL0"
 		(at 186.69 38.1 0)
 		(effects
@@
 		)
 	)
-	(label "GPIO1"
-		(at 52.07 43.18 0)
-		(effects
-			(font
-				(size 1.27 1.27)
-			)
-			(justify left bottom)
-		)
-	)
 	(label "I2C_SDA"
 		(at 121.92 99.06 0)
@@
 		)
 	)
-	(label "GPIO3"
+	(label "ENET_TXEN"
 		(at 189.23 91.44 0)
 		(effects
@@
 		)
 	)
-	(label "GPIO4"
+	(label "GPIO7"
 		(at 186.69 129.54 0)
 		(effects
@@
 		)
 	)
-	(label "PWM0"
-		(at 100.33 33.02 0)
-		(effects
-			(font
-				(size 1.27 1.27)
-			)
-			(justify left bottom)
-		)
-	)
-	(label "PWM3"
+	(label "PWM4"
 		(at 186.69 40.64 0)
 		(effects
@@
 		)
 	)
-	(label "PWM0"
+	(label "PWM3"
 		(at 186.69 30.48 0)
 		(effects
@@
 		)
 	)
-	(label "GPIO2"
+	(label "ENET_RXD1"
 		(at 189.23 88.9 0)
 		(effects
@@
 		)
 	)
-	(label "GPIO3"
-		(at 52.07 38.1 0)
-		(effects
-			(font
-				(size 1.27 1.27)
-			)
-			(justify left bottom)
-		)
-	)
 	(label "M1-"
 		(at 224.79 35.56 0)
@@
 		)
 	)
-	(label "GPIO2"
-		(at 52.07 45.72 0)
-		(effects
-			(font
-				(size 1.27 1.27)
-			)
-			(justify left bottom)
-		)
-	)
-	(label "GPIO0"
+	(label "T_COL0"
 		(at 186.69 25.4 0)
 		(effects
@@
 		)
 	)
-	(label "GPIO4"
-		(at 52.07 40.64 0)
-		(effects
-			(font
-				(size 1.27 1.27)
-			)
-			(justify left bottom)
-		)
-	)
-	(label "GPIO0"
-		(at 52.07 50.8 0)
-		(effects
-			(font
-				(size 1.27 1.27)
-			)
-			(justify left bottom)
-		)
-	)
 	(label "I2C_SCL"
 		(at 100.33 71.12 0)
@@
 			)
 		)
-		(property "Footprint" "Connector_PinHeader_2.54mm:PinHeader_1x10_P2.54mm_Vertical"
+		(property "Footprint" "Connector_PinHeader_2.54mm:PinHeader_1x12_P2.54mm_Vertical"
 			(at 209.55 54.61 0)
 			(hide yes)
